File: Christmas.kicad_sch (KiCad schematic)
At the start: 13 parts

Commit message: final improvements to V0.1 of pcb
-improved silkscreen
Other:
- title: Christmas light -> Christmas PCB tree
Changed lines of the file:
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@@
   (paper "A5")
   (title_block
-    (title "Christmas light")
-    (date "2023-12-05")
+    (title "Christmas PCB tree")
+    (date "2023-12-06")
     (rev "V0.2")
+    (comment 1 "Casper Tak")
   )
   (junction (at 134.62 64.77) (diameter 0) (color 0 0 0 0)
